File: pcb/banjobox/banjobox.kicad_sch (KiCad schematic)
At the start: 0 parts

Commit message: rearranged files
Parts:
- added C1: 1uF, symbol Device:C_Polarized
- added C2: 10uf, symbol Device:C_Polarized
- added C3: 0.1uF, symbol Device:C
- added C4, C5: 100nF, symbol Device:C
- added C6: 10uF, symbol Device:C_Polarized
- added C7: 100uF, symbol Device:C_Polarized
- added LS1: Speaker, symbol Device:Speaker
- added R1, R2: 4.7k, symbol Device:R
- added R3: 100k, symbol Device:R
- added RV1: 10K, symbol Device:R_Potentiometer_Trim
- added SW1: RotaryEncoder_Switch, symbol Device:RotaryEncoder_Switch
- added U1: SHT31-DIS, Sensor_Humidity:Sensirion_DFN-8-1EP_2.5x2.5mm_P0.5mm_EP1.1x1.7mm, symbol Sensor_Humidity:SHT31-DIS
- added U2: MOUDLE-SEEEDUINO-XIAO, symbol XIAO_RP2040:MOUDLE-SEEEDUINO-XIAO
- added U3: ER_OLEDM0.91_1x-I2C, Display:ER_OLEDM0.91_1x-I2C, symbol Display_Graphic:ER_OLEDM0.91_1x-I2C
- added U4: PAM8302AAY, Package_DFN_QFN:DFN-8-1EP_3x3mm_P0.65mm_EP1.55x2.4mm, symbol Amplifier_Audio:PAM8302AAY
Connections:
- new net: C3.2, RV1.1
- new net: RV1.2, U4.3 (IN+)
- new net: LS1.1, U4.5 (OUT+)
- new net: LS1.2, U4.8 (OUT-)
- new net EC11A: SW1.A, U2.1 (PA02_A0_D0)
- new net EC11B: SW1.B, U2.2 (PA4_A1_D1)
- new net EC11SW1: SW1.S1, U2.3 (PA10_A2_D2)
- new net GND: C1.2, C2.2, C4.1, C5.1, C6.2, C7.2, R3.2, RV1.3, SW1.C, SW1.S2, U1.2 (ADDR), U1.7 (R), U1.8 (VSS), U1.9 (VSS), U2.13 (GND), U3.1 (GND), U4.4 (IN-), U4.7 (GND)
- new net PWM: C3.1, R3.1, U2.4 (PA11_A3_D3)
- new net SCL: R2.1, U1.4 (SCL), U2.6 (PA9_A5_D5_SCL), U3.3 (SCL)
- new net SDA: R1.2, U1.1 (SDA), U2.5 (PA8_A4_D4_SDA), U3.4 (SDA)
- new net VCC: C1.1, C2.1, C4.2, C5.2, C6.1, C7.1, R1.1, R2.2, U1.5 (VDD), U2.12 (3V3), U3.2 (VCC), U4.6 (VDD)
- no-connect marks 0 -> 1
Other:
- note added: "Amplifier and speaker"
- note added: "Encoder"
- note added: "OLED display"
- note added: "Temp/ Humidity sensor"
- title: (none) -> Banjobox
